File: hw/simm/breakout/simm72_breakout.kicad_sch (KiCad schematic)
At the start: 5 parts, among them J1 SIMM72, J2 Conn_02x08_Row_Letter_Last, J3 Conn_02x08_Row_Letter_Last, J4 Conn_02x08_Row_Letter_Last, J5 Conn_02x08_Row_Letter_Last

Commit message: simm folder cleanup and license
Other:
- company: www.happydaze.se -> Licensed under CERN-OHL-P v2
Changed lines of the file:
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@@
     (date "2023")
     (rev "A0")
-    (company "www.happydaze.se")
+    (company "Licensed under CERN-OHL-P v2")
+    (comment 1 "Anders Granlund")
+    (comment 4 "PCB depth : 1.2mm")
   )
   (junction (at 55.245 137.16) (diameter 0) (color 0 0 0 0)
@@
     (pin "9")
     (instances
-      (project "simm72"
+      (project "simm72_breakout"
         (path "/0981ba96-97e1-483d-834d-af22b04cbe88"
           (reference "J1") (unit 1)
@@
     (pin "14")
     (instances
-      (project "simm72"
+      (project "simm72_breakout"
         (path "/0981ba96-97e1-483d-834d-af22b04cbe88"
           (reference "J2") (unit 1)
@@
     (pin "1")
     (instances
-      (project "simm72"
+      (project "simm72_breakout"
         (path "/0981ba96-97e1-483d-834d-af22b04cbe88"
           (reference "#PWR04") (unit 1)
@@
     (pin "1")
     (instances
-      (project "simm72"
+      (project "simm72_breakout"
         (path "/0981ba96-97e1-483d-834d-af22b04cbe88"
           (reference "#PWR02") (unit 1)
@@
     (pin "1")
     (instances
-      (project "simm72"
+      (project "simm72_breakout"
         (path "/0981ba96-97e1-483d-834d-af22b04cbe88"
           (reference "#PWR01") (unit 1)
@@
     (pin "9")
     (instances
-      (project "simm72"
+      (project "simm72_breakout"
         (path "/0981ba96-97e1-483d-834d-af22b04cbe88"
           (reference "J3") (unit 1)
@@
     (pin "9")
     (instances
-      (project "simm72"
+      (project "simm72_breakout"
         (path "/0981ba96-97e1-483d-834d-af22b04cbe88"
           (reference "J5") (unit 1)
@@
     (pin "1")
     (instances
-      (project "simm72"
+      (project "simm72_breakout"
         (path "/0981ba96-97e1-483d-834d-af22b04cbe88"
           (reference "#PWR03") (unit 1)
@@
     (pin "5")
     (instances
-      (project "simm72"
+      (project "simm72_breakout"
         (path "/0981ba96-97e1-483d-834d-af22b04cbe88"
           (reference "J4") (unit 1)
@@
     (pin "1")
     (instances
-      (project "simm72"
+      (project "simm72_breakout"
         (path "/0981ba96-97e1-483d-834d-af22b04cbe88"
           (reference "#PWR05") (unit 1)
