File: hw/simm/ram_16M55/simm72_ram_16M55.kicad_sch (KiCad schematic)
At the start: 5 parts, among them IC1 AS6C6416-55TIN, IC2 AS6C6416-55TIN, J1 SIMM72

Commit message: simm folder cleanup and license
Other:
- company: www.happydaze.se -> Licensed under CERN-OHL-P v2
Changed lines of the file:
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@@
     (date "2023")
     (rev "A0")
-    (company "www.happydaze.se")
+    (company "Licensed under CERN-OHL-P v2")
+    (comment 1 "Anders Granlund")
   )
   (junction (at 172.085 33.02) (diameter 0) (color 0 0 0 0)
@@
     (pin "9")
     (instances
-      (project "simm72"
+      (project "simm72_ram_16M55"
         (path "/0981ba96-97e1-483d-834d-af22b04cbe88"
           (reference "J1") (unit 1)
@@
     (pin "1")
     (instances
-      (project "simm72"
+      (project "simm72_ram_16M55"
         (path "/0981ba96-97e1-483d-834d-af22b04cbe88"
           (reference "#PWR014") (unit 1)
@@
     (pin "1")
     (instances
-      (project "simm72"
+      (project "simm72_ram_16M55"
         (path "/0981ba96-97e1-483d-834d-af22b04cbe88"
           (reference "#PWR04") (unit 1)
@@
     (pin "1")
     (instances
-      (project "simm72"
+      (project "simm72_ram_16M55"
         (path "/0981ba96-97e1-483d-834d-af22b04cbe88"
           (reference "#PWR09") (unit 1)
@@
     (pin "1")
     (instances
-      (project "simm72"
+      (project "simm72_ram_16M55"
         (path "/0981ba96-97e1-483d-834d-af22b04cbe88"
           (reference "#PWR02") (unit 1)
@@
     (pin "29")
     (instances
-      (project "simm72"
+      (project "simm72_ram_16M55"
         (path "/0981ba96-97e1-483d-834d-af22b04cbe88"
           (reference "IC1") (unit 1)
@@
     (pin "1")
     (instances
-      (project "simm72"
+      (project "simm72_ram_16M55"
         (path "/0981ba96-97e1-483d-834d-af22b04cbe88"
           (reference "#PWR01") (unit 1)
@@
     (pin "1")
     (instances
-      (project "simm72"
+      (project "simm72_ram_16M55"
         (path "/0981ba96-97e1-483d-834d-af22b04cbe88"
           (reference "#PWR07") (unit 1)
@@
     (pin "1")
     (instances
-      (project "simm72"
+      (project "simm72_ram_16M55"
         (path "/0981ba96-97e1-483d-834d-af22b04cbe88"
           (reference "#PWR010") (unit 1)
@@
     (pin "29")
     (instances
-      (project "simm72"
+      (project "simm72_ram_16M55"
         (path "/0981ba96-97e1-483d-834d-af22b04cbe88"
           (reference "IC2") (unit 1)
@@
     (pin "1")
     (instances
-      (project "simm72"
+      (project "simm72_ram_16M55"
         (path "/0981ba96-97e1-483d-834d-af22b04cbe88"
           (reference "#PWR08") (unit 1)
@@
     (pin "1")
     (instances
-      (project "simm72"
+      (project "simm72_ram_16M55"
         (path "/0981ba96-97e1-483d-834d-af22b04cbe88"
           (reference "#PWR013") (unit 1)
@@
     (pin "1")
     (instances
-      (project "simm72"
+      (project "simm72_ram_16M55"
         (path "/0981ba96-97e1-483d-834d-af22b04cbe88"
           (reference "#PWR011") (unit 1)
@@
     (pin "1")
     (instances
-      (project "simm72"
+      (project "simm72_ram_16M55"
         (path "/0981ba96-97e1-483d-834d-af22b04cbe88"
           (reference "#PWR06") (unit 1)
@@
     (pin "1")
     (instances
-      (project "simm72"
+      (project "simm72_ram_16M55"
         (path "/0981ba96-97e1-483d-834d-af22b04cbe88"
           (reference "#PWR05") (unit 1)
@@
     (pin "1")
     (instances
-      (project "simm72"
+      (project "simm72_ram_16M55"
         (path "/0981ba96-97e1-483d-834d-af22b04cbe88"
           (reference "C2") (unit 1)
@@
     (pin "1")
     (instances
-      (project "simm72"
+      (project "simm72_ram_16M55"
         (path "/0981ba96-97e1-483d-834d-af22b04cbe88"
           (reference "#PWR03") (unit 1)
@@
     (pin "1")
     (instances
-      (project "simm72"
+      (project "simm72_ram_16M55"
         (path "/0981ba96-97e1-483d-834d-af22b04cbe88"
           (reference "C1") (unit 1)
@@
     (pin "1")
     (instances
-      (project "simm72"
+      (project "simm72_ram_16M55"
         (path "/0981ba96-97e1-483d-834d-af22b04cbe88"
           (reference "#PWR012") (unit 1)
