File: hw/simm/ram_8M10/simm72_ram_8M10.kicad_sch (KiCad schematic)
At the start: 7 parts, among them IC1 IS61WV204816BLL-10TLI, IC2 IS61WV204816BLL-10TLI, J1 SIMM72

Commit message: simm folder cleanup and license
Other:
- company: www.happydaze.se -> Licensed under CERN-OHL-P v2
Changed lines of the file:
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@@
     (date "2023")
     (rev "A0")
-    (company "www.happydaze.se")
+    (company "Licensed under CERN-OHL-P v2")
+    (comment 1 "Anders Granlund")
   )
   (junction (at 193.04 53.34) (diameter 0) (color 0 0 0 0)
