File: hw/simm/rom_2M55/simm72_rom_2M55.kicad_sch (KiCad schematic)
At the start: 9 parts, among them J1 SIMM72, U1 SST39LF040, U2 SST39LF040, U3 SST39LF040, U4 SST39LF040

Commit message: simm folder cleanup and license
Other:
- company: www.happydaze.se -> Licensed under CERN-OHL-P v2
Changed lines of the file:
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@@
     (date "2023")
     (rev "A0")
-    (company "www.happydaze.se")
+    (company "Licensed under CERN-OHL-P v2")
+    (comment 1 "Anders Granlund")
   )
   (junction (at 119.38 147.32) (diameter 0) (color 0 0 0 0)
