File: hw/simm/template/simm72.kicad_sch (KiCad schematic)
At the start: 1 part, among them J1 SIMM72

Commit message: simm folder cleanup and license
Other:
- company: www.happydaze.se -> (none)
- title: Raven SIMM template -> (none)
Changed lines of the file:
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@@
 (kicad_sch (version 20230121) (generator eeschema)
   (paper "A4")
-  (title_block
-    (title "Raven SIMM template")
-    (date "2023")
-    (rev "A0")
-    (company "www.happydaze.se")
-  )
   (junction (at 55.245 137.16) (diameter 0) (color 0 0 0 0)
   )
