File: hw/isa/template_16bit/isa16.kicad_sch (KiCad schematic)
At the start: 1 part, among them J1 ISA16_Edge

Commit message: isa folder cleanup
Other:
- title: ISA Template 16bit -> (none)
Changed lines of the file:
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@@
 (kicad_sch (version 20230121) (generator eeschema)
   (paper "A3")
-  (title_block
-    (title "ISA Template 16bit")
-  )
   (symbol (lib_id "68k:ISA16_Edge") (at 71.12 133.35 0) (unit 1)
     (in_bom yes) (on_board yes) (dnp no)
