File: hw/raven/a1/misc.kicad_sch (KiCad schematic)
At the start: 53 parts, among them J204 PinHdr_01x04, J401 DB25/9/9, J601 TRSx2, J606 DB9M/9M, J607 PS/2 (dual), U601 CNY17F-3, U602 74LS07

Commit message: fixed bom error
Parts:
- J204: Manufacturer_Part_Number 61300211021 -> 61300411121
Changed lines of the file:
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@@
       (effects (font (size 1.27 1.27)) hide)
     )
-    (property "Manufacturer_Part_Number" "61300211021" (at 346.71 60.96 0)
+    (property "Manufacturer_Part_Number" "61300411121" (at 346.71 60.96 0)
       (effects (font (size 1.27 1.27)) hide)
     )
@@
       (effects (font (size 1.27 1.27)) hide)
     )
-    (property "Manufacturer_Part_Number" "61300211021" (at 331.47 86.995 0)
+    (property "Manufacturer_Part_Number" "61300411121" (at 331.47 86.995 0)
       (effects (font (size 1.27 1.27)) hide)
     )
@@
       (effects (font (size 1.27 1.27)) hide)
     )
-    (property "Manufacturer_Part_Number" "61300211021" (at 331.47 60.96 0)
-      (effects (font (size 1.27 1.27)) hide)
-    )
+    (property "Manufacturer_Part_Number" "61300411121" (at 331.47 60.96 0)
+      (effects (font (size 1.27 1.27)) hide)
+    )
