File: hw/simm/rom_2M55_PLCC/simm72_rom_2M55.kicad_sch (KiCad schematic)
At the start: 9 parts, among them J1 SIMM72, U1 SST39LF040, U2 SST39LF040, U3 SST39LF040, U4 SST39LF040

Commit message: Changed ROM Simm naming convention
Other:
- title: Raven flash rom -> Raven 2MB ROM
Changed lines of the file:
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@@
   (paper "A4")
   (title_block
-    (title "Raven flash rom")
+    (title "Raven 2MB ROM")
     (date "2023")
     (rev "A0")
