File: hw/raven/a2/power.kicad_sch (KiCad schematic)
At the start: 28 parts, among them J1 ATX Power, J202 Pinhdr_02x05, J203 Pinhdr_01x03, J305 FanHeader, SW201 SW_Push, SW202 SW_Push, U201 LM7905CT_NOPB, U202 MAX16054AZT+T, U203 DS1818, U204 74HCT10

Commit message: Rev.A2 some minor fixes
Parts:
- SW201, SW202: Manufacturer_Part_Number SKHHARA010 -> SKHHAKA010
Changed lines of the file:
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@@
       (effects (font (size 1.27 1.27)) hide)
     )
-    (property "Manufacturer_Part_Number" "SKHHARA010" (at 80.645 123.825 0)
+    (property "Manufacturer_Part_Number" "SKHHAKA010" (at 80.645 123.825 0)
       (effects (font (size 1.27 1.27)) hide)
     )
@@
       (effects (font (size 1.27 1.27)) hide)
     )
-    (property "Manufacturer_Part_Number" "SKHHARA010" (at 44.45 51.435 0)
-      (effects (font (size 1.27 1.27)) hide)
-    )
+    (property "Manufacturer_Part_Number" "SKHHAKA010" (at 44.45 51.435 0)
+      (effects (font (size 1.27 1.27)) hide)
+    )

Commit message: A2 : minor changes to aid in building
Silkscreen improvements
Larger diode footprints
Parts:
- D1, D2, D3: footprint Diode_SMD:D_SOD-123F -> 68k:D_SOD-123F_Handsolder
Changed lines of the file:
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@@
       (effects (font (size 1.27 1.27)))
     )
-    (property "Footprint" "Diode_SMD:D_SOD-123F" (at 254.635 86.36 0)
+    (property "Footprint" "68k:D_SOD-123F_Handsolder" (at 254.635 86.36 0)
       (effects (font (size 1.27 1.27)) hide)
     )
@@
       (effects (font (size 1.27 1.27)))
     )
-    (property "Footprint" "Diode_SMD:D_SOD-123F" (at 263.525 86.36 0)
+    (property "Footprint" "68k:D_SOD-123F_Handsolder" (at 263.525 86.36 0)
       (effects (font (size 1.27 1.27)) hide)
     )
@@
       (effects (font (size 1.27 1.27)))
     )
-    (property "Footprint" "Diode_SMD:D_SOD-123F" (at 245.745 86.36 0)
-      (effects (font (size 1.27 1.27)) hide)
-    )
+    (property "Footprint" "68k:D_SOD-123F_Handsolder" (at 245.745 86.36 0)
+      (effects (font (size 1.27 1.27)) hide)
+    )
