File: hw/raven/a2/local32.kicad_sch (KiCad schematic)
At the start: 98 parts, among them J301 SIMM72, J302 SIMM72, J303 SIMM72, J304 SIMM72, J305 PWM, J306 USB2Header, J307 ARGB, J308 ESSI1, U301 CH559L, U302 CH213K, U303 XR68M752, U304 MAX3245CAI+T, U305 DSP56303, U306 PCM180PW, U307 AS7C31024B-xxTJ, U308 AS7C31024B-xxTJ, U309 AS7C31024B-xxTJ, U310 SN74LVC1G14DBV, U311 PCM5102A, X301 ASE-24.000MHZ-L-C-T, X302 ASELJ-E-22.5792MHz

Commit message: cosmetic
Changed lines of the file:
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@@
 	(text_box "todo:\n? i2c on P1.2, P1.3\n - for ikbd rtc without need for software driver\n - for eiffel-lcd support\n - generic uart<->i2c interface\n\n? spi on p1.4, p1.5, p.16\n - plus suitable CS pins (2 or so)\n - routed to spi header(s) on motherboard\n - generic uart<->spi interface\n"
 		(exclude_from_sim no)
-		(at 318.77 100.965 0)
+		(at 331.47 99.06 0)
 		(size 46.99 26.035)
 		(margins 0.9525 0.9525 0.9525 0.9525)
@@
 	)
 	(junction
-		(at 790.575 491.49)
+		(at 790.575 488.95)
 		(diameter 0)
 		(color 0 0 0 0)
@@
 	)
 	(junction
-		(at 798.195 491.49)
+		(at 798.195 488.95)
 		(diameter 0)
 		(color 0 0 0 0)
@@
 	)
 	(junction
+		(at 806.45 488.95)
+		(diameter 0)
+		(color 0 0 0 0)
+	)
+	(junction
 		(at 537.21 484.505)
 		(diameter 0)
@@
 	(wire
 		(pts
-			(xy 806.45 491.49) (xy 798.195 491.49)
+			(xy 806.45 488.95) (xy 798.195 488.95)
 		)
 		(stroke
@@
 	(wire
 		(pts
-			(xy 782.955 486.41) (xy 782.955 491.49)
+			(xy 782.955 486.41) (xy 782.955 488.95)
 		)
 		(stroke
@@
 	(wire
 		(pts
-			(xy 798.195 486.41) (xy 798.195 491.49)
+			(xy 798.195 486.41) (xy 798.195 488.95)
 		)
 		(stroke
@@
 	(wire
 		(pts
-			(xy 782.955 491.49) (xy 790.575 491.49)
+			(xy 782.955 488.95) (xy 790.575 488.95)
 		)
 		(stroke
@@
 	(wire
 		(pts
-			(xy 790.575 486.41) (xy 790.575 491.49)
+			(xy 790.575 486.41) (xy 790.575 488.95)
 		)
 		(stroke
@@
 	(wire
 		(pts
-			(xy 806.45 486.41) (xy 806.45 491.49)
+			(xy 806.45 486.41) (xy 806.45 488.95)
 		)
 		(stroke
@@
 	(wire
 		(pts
-			(xy 798.195 491.49) (xy 798.195 493.395)
+			(xy 806.45 488.95) (xy 806.45 490.855)
 		)
 		(stroke
@@
 	(wire
 		(pts
-			(xy 790.575 491.49) (xy 798.195 491.49)
+			(xy 790.575 488.95) (xy 798.195 488.95)
 		)
 		(stroke
@@
 		(dnp no)
 		(property "Reference" "C334"
-			(at 368.3 440.69 90)
+			(at 369.062 440.69 90)
 			(effects
 				(font
@@
 		(dnp no)
 		(property "Reference" "C341"
-			(at 796.544 487.68 90)
+			(at 801.116 482.092 0)
 			(effects
 				(font
@@
 		)
 		(property "Value" "0.1u"
-			(at 799.846 487.426 90)
+			(at 800.862 485.902 0)
 			(effects
 				(font
@@
 	(symbol
 		(lib_id "power:GND")
-		(at 798.195 493.395 0)
+		(at 806.45 490.855 0)
 		(unit 1)
 		(exclude_from_sim no)
@@
 		(dnp no)
 		(fields_autoplaced yes)
-		(property "Reference" "#PWR0400"
-			(at 798.195 499.745 0)
+		(property "Reference" "#PWR0398"
+			(at 806.45 497.205 0)
 			(effects
 				(font
@@
 		)
 		(property "Value" "GND"
-			(at 798.195 498.475 0)
+			(at 806.45 495.935 0)
 			(effects
 				(font
@@
 		)
 		(property "Footprint" ""
-			(at 798.195 493.395 0)
+			(at 806.45 490.855 0)
 			(effects
 				(font
@@
 		)
 		(property "Datasheet" ""
-			(at 798.195 493.395 0)
+			(at 806.45 490.855 0)
 			(effects
 				(font
@@
 		)
 		(property "Description" ""
-			(at 798.195 493.395 0)
+			(at 806.45 490.855 0)
 			(effects
 				(font
@@
 			(project "raven"
 				(path "/af55e73e-5814-45b4-ac5c-0bab62c0b1c7/d5022d96-0fa0-4474-b160-b3a99bf8c2e1"
-					(reference "#PWR0400")
+					(reference "#PWR0398")
 					(unit 1)
 				)
@@
 		(dnp no)
 		(property "Reference" "C333"
-			(at 770.763 395.732 90)
+			(at 770.636 393.7 0)
 			(effects
 				(font
@@
 		)
 		(property "Value" "1u"
-			(at 764.921 395.732 90)
+			(at 769.366 397.764 0)
 			(effects
 				(font
@@
 		(dnp no)
 		(property "Reference" "C332"
-			(at 759.714 395.351 90)
+			(at 759.714 393.954 0)
 			(effects
 				(font
@@
 		)
 		(property "Value" "0.1u"
-			(at 754.126 395.351 90)
+			(at 759.46 397.51 0)
 			(effects
 				(font
@@
 		(on_board yes)
 		(dnp no)
-		(property "Reference" "#PWR0398"
+		(property "Reference" "#PWR0399"
 			(at 528.32 499.745 0)
 			(effects
@@
 			(project "raven"
 				(path "/af55e73e-5814-45b4-ac5c-0bab62c0b1c7/d5022d96-0fa0-4474-b160-b3a99bf8c2e1"
-					(reference "#PWR0398")
+					(reference "#PWR0399")
 					(unit 1)
 				)
@@
 		(dnp no)
 		(property "Reference" "C303"
-			(at 690.245 222.631 90)
+			(at 690.372 216.916 90)
 			(effects
 				(font
@@
 		)
 		(property "Value" "10u"
-			(at 690.245 217.17 90)
+			(at 690.118 222.758 90)
 			(effects
 				(font
@@
 		(on_board yes)
 		(dnp no)
-		(property "Reference" "#PWR0399"
+		(property "Reference" "#PWR0400"
 			(at 530.86 499.745 0)
 			(effects
@@
 			(project "raven"
 				(path "/af55e73e-5814-45b4-ac5c-0bab62c0b1c7/d5022d96-0fa0-4474-b160-b3a99bf8c2e1"
-					(reference "#PWR0399")
+					(reference "#PWR0400")
 					(unit 1)
 				)
@@
 		(dnp no)
 		(property "Reference" "C342"
-			(at 805.18 487.426 90)
+			(at 809.498 482.092 0)
 			(effects
 				(font
@@
 		)
 		(property "Value" "1u"
-			(at 808.228 486.664 90)
+			(at 808.228 485.902 0)
 			(effects
 				(font
@@
 		)
 		(property "Value" "+5V"
-			(at 564.515 241.935 0)
+			(at 563.372 242.062 90)
 			(effects
 				(font
@@
 		(dnp no)
 		(property "Reference" "C339"
-			(at 781.304 487.68 90)
+			(at 785.876 482.092 0)
 			(effects
 				(font
@@
 		)
 		(property "Value" "0.1u"
-			(at 784.352 487.172 90)
+			(at 785.368 485.902 0)
 			(effects
 				(font
@@
 		(dnp no)
 		(property "Reference" "C331"
-			(at 723.392 395.478 90)
+			(at 723.138 389.636 90)
 			(effects
 				(font
@@
 		)
 		(property "Value" "0.1u"
-			(at 723.138 389.89 90)
+			(at 723.138 395.478 90)
 			(effects
 				(font
@@
 		(dnp no)
 		(property "Reference" "C340"
-			(at 788.924 487.426 90)
+			(at 793.496 482.092 0)
 			(effects
 				(font
@@
 		)
 		(property "Value" "0.1u"
-			(at 792.226 486.918 90)
+			(at 793.242 485.902 0)
 			(effects
 				(font

Commit message: A2: cosmetics and bom preparations
Parts:
- C305: footprint Capacitor_THT:CP_Radial_D5.0mm_P2.50mm -> Capacitor_THT:CP_Radial_D6.3mm_P2.50mm; Manufacturer_Part_Number EEU-EB1H100SH -> ECE-A1HKS100I
- C306: footprint Capacitor_THT:CP_Radial_D5.0mm_P2.50mm -> Capacitor_THT:CP_Radial_D6.3mm_P2.50mm; Manufacturer_Part_Number EEU-EB1A101SH -> ECE-A1AKS101
- J305: value PWM -> FanHeader
- J306: value USB2Header -> PinHdr_02x05
- J307: value ARGB -> FanHeader
- J308: value ESSI1 -> PinHdr_02x05; Manufacturer_Part_Number (none) -> 61201021621; Manufacturer_Part_Numer 61201021621 -> (none)
- U304: value MAX3245CAI+T -> MAX3245
- U306: value PCM180PW -> PCM1808
- U307, U308, U309: value AS7C31024B-xxTJ -> AS7C31024B
- U310: value SN74LVC1G14DBV -> SN74LVC1G14
- X301: value ASE-24.000MHZ-L-C-T -> 24Mhz (3.3V); Manufacturer_Name ABRACON -> Abracon
- X302: value ASELJ-E-22.5792MHz -> 22.5792MHz (3.3V); Manufacturer_Name ABRACON -> Abracon
