File: hw/raven/a2/local16.kicad_sch (KiCad schematic)
At the start: 34 parts, among them J401 IDE44, J402 BatteryHolder, U401 MC68901, U402 ATF22V10C-10PU, U403 MC68901, U404 MAX3245CAI+T, U405 YM2149, U406 DS1307, U407 24AA02E48, X401 8Mhz (5V)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

Commit message: A2 routing
Parts:
- added C413: 1u, Capacitor_SMD:C_1206_3216Metric_Pad1.33x1.80mm_HandSolder, symbol 68k:c_100nf_smd1206
- renumbered C413 to C414, C414 to C415
Connections:
- net +5V: now also U403.26 (I4)
- net +5VL: now also C413.2
- net GND: now also C413.1
- no-connect marks 21 -> 20
Other:
- note added: "blitter/dsp"
- note removed: "blitter irq"

Commit message: A2: schema + routing complete. ERC + DRC complete.
Let sit for a while, revisit and sanity check with fresh eyes before gerber.
Todo: double check BOM export and fix missing infos if any.
Parts:
- added R405: 2K2, Resistor_SMD:R_1206_3216Metric_Pad1.30x1.75mm_HandSolder, symbol Device:R
- renumbered R405 to R406, R406 to R407, R407 to R408, R408 to R409
Connections:
- net +5V: now also R405.1; no longer U403.26 (I4)
- net ~{IRQ_VBL} renamed MFP2:TCO
- new net: R405.2, U403.26 (I4)
- no-connect marks 20 -> 21
Changed lines of the file:
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@@
 		)
 	)
-	(text_box "TODO:\nConnect one of TxO directly to IRQ4 (VBLANK)\nOne of TxO could be used for buzzer"
-		(exclude_from_sim no)
-		(at 514.35 45.72 0)
-		(size 50.8 10.16)
-		(margins 0.9525 0.9525 0.9525 0.9525)
-		(stroke
-			(width 0)
-			(type solid)
-		)
-		(fill
-			(type color)
-			(color 255 230 63 0.53)
-		)
-		(effects
-			(font
-				(size 1.27 1.27)
-				(color 0 0 0 1)
-			)
-			(justify left top)
-		)
-	)
 	(text_box ""
 		(exclude_from_sim no)
@@
 	)
 	(no_connect
+		(at 492.76 78.74)
+	)
+	(no_connect
 		(at 92.71 217.805)
 	)
@@
 	(wire
 		(pts
-			(xy 471.805 78.74) (xy 493.395 78.74)
-		)
-		(stroke
-			(width 0)
-			(type default)
-		)
-	)
-	(wire
-		(pts
 			(xy 287.655 92.71) (xy 287.655 97.79)
 		)
@@
 	(wire
 		(pts
+			(xy 471.805 78.74) (xy 492.76 78.74)
+		)
+		(stroke
+			(width 0)
+			(type default)
+		)
+	)
+	(wire
+		(pts
 			(xy 178.435 189.865) (xy 189.23 189.865)
 		)
@@
 	(wire
 		(pts
+			(xy 359.41 43.18) (xy 359.41 44.45)
+		)
+		(stroke
+			(width 0)
+			(type default)
+		)
+	)
+	(wire
+		(pts
 			(xy 227.965 97.79) (xy 241.935 97.79)
 		)
@@
 	(wire
 		(pts
+			(xy 359.41 64.77) (xy 287.655 64.77)
+		)
+		(stroke
+			(width 0)
+			(type default)
+		)
+	)
+	(wire
+		(pts
 			(xy 467.995 119.38) (xy 470.535 119.38)
 		)
@@
 	(wire
 		(pts
-			(xy 287.655 64.77) (xy 346.075 64.77)
-		)
-		(stroke
-			(width 0)
-			(type default)
-		)
-	)
-	(wire
-		(pts
 			(xy 441.96 193.04) (xy 445.77 193.04)
 		)
@@
 	(wire
 		(pts
+			(xy 359.41 52.07) (xy 359.41 64.77)
+		)
+		(stroke
+			(width 0)
+			(type default)
+		)
+	)
+	(wire
+		(pts
 			(xy 156.21 206.375) (xy 161.925 206.375)
 		)
@@
 		)
 	)
-	(global_label "~{IRQ_VBL}"
-		(shape output)
-		(at 493.395 78.74 0)
-		(fields_autoplaced yes)
-		(effects
-			(font
-				(size 1.27 1.27)
-			)
-			(justify left)
-		)
-		(property "Intersheetrefs" "${INTERSHEET_REFS}"
-			(at 503.9398 78.74 0)
-			(effects
-				(font
-					(size 1.27 1.27)
-				)
-				(justify left)
-				(hide yes)
-			)
-		)
-	)
 	(global_label "LPT1:~{BUSY}"
 		(shape input)
@@
 		(on_board yes)
 		(dnp no)
-		(property "Reference" "R407"
+		(property "Reference" "R408"
 			(at 48.26 207.645 90)
 			(effects
@@
 			(project "raven"
 				(path "/af55e73e-5814-45b4-ac5c-0bab62c0b1c7/dacbbff1-3783-4e73-aa71-dbe41700eceb"
-					(reference "R407")
+					(reference "R408")
 					(unit 1)
 				)
@@
 		(on_board yes)
 		(dnp no)
-		(property "Reference" "#PWR0416"
+		(property "Reference" "#PWR0417"
 			(at 56.515 60.325 0)
 			(effects
@@
 			(project "raven"
 				(path "/af55e73e-5814-45b4-ac5c-0bab62c0b1c7/dacbbff1-3783-4e73-aa71-dbe41700eceb"
-					(reference "#PWR0416")
+					(reference "#PWR0417")
 					(unit 1)
 				)
@@
 		(on_board yes)
 		(dnp no)
-		(property "Reference" "#PWR0417"
+		(property "Reference" "#PWR0418"
 			(at 211.455 70.485 0)
 			(effects
@@
 			(project "raven"
 				(path "/af55e73e-5814-45b4-ac5c-0bab62c0b1c7/dacbbff1-3783-4e73-aa71-dbe41700eceb"
-					(reference "#PWR0417")
+					(reference "#PWR0418")
 					(unit 1)
 				)
@@
 		(on_board yes)
 		(dnp no)
-		(property "Reference" "R405"
+		(property "Reference" "R406"
 			(at 39.37 193.675 90)
 			(effects
@@
 			(project "raven"
 				(path "/af55e73e-5814-45b4-ac5c-0bab62c0b1c7/dacbbff1-3783-4e73-aa71-dbe41700eceb"
-					(reference "R405")
+					(reference "R406")
 					(unit 1)
 				)
@@
 			)
 		)
-		(property "Datasheet" ""
+		(property "Datasheet" "http://cdn-reichelt.de/documents/datenblatt/B400/OSZI.pdf"
 			(at 53.975 65.405 0)
 			(effects
@@
 			)
 		)
-		(property "Description" ""
+		(property "Description" "Crystal Clock Oscillator, DIP8-style metal package"
 			(at 56.515 65.405 0)
 			(effects
@@
 					(size 1.27 1.27)
 				)
+				(hide yes)
 			)
 		)
@@
 	(symbol
 		(lib_id "power:+5V")
-		(at 346.075 64.77 270)
+		(at 359.41 43.18 0)
 		(unit 1)
 		(exclude_from_sim no)
@@
 		(on_board yes)
 		(dnp no)
-		(property "Reference" "#PWR0418"
-			(at 342.265 64.77 0)
+		(property "Reference" "#PWR0416"
+			(at 359.41 46.99 0)
 			(effects
 				(font
@@
 		)
 		(property "Value" "+5V"
-			(at 351.028 64.77 90)
+			(at 359.41 39.116 0)
 			(effects
 				(font
@@
 		)
 		(property "Footprint" ""
-			(at 346.075 64.77 0)
+			(at 359.41 43.18 0)
 			(effects
 				(font
@@
 		)
 		(property "Datasheet" ""
-			(at 346.075 64.77 0)
+			(at 359.41 43.18 0)
 			(effects
 				(font
@@
 		)
 		(property "Description" ""
-			(at 346.075 64.77 0)
+			(at 359.41 43.18 0)
 			(effects
 				(font
@@
 			(project "raven"
 				(path "/af55e73e-5814-45b4-ac5c-0bab62c0b1c7/dacbbff1-3783-4e73-aa71-dbe41700eceb"
-					(reference "#PWR0418")
+					(reference "#PWR0416")
 					(unit 1)
 				)
@@
 		(on_board yes)
 		(dnp no)
-		(property "Reference" "R406"
+		(property "Reference" "R407"
 			(at 28.575 208.28 90)
 			(effects
@@
 			(project "raven"
 				(path "/af55e73e-5814-45b4-ac5c-0bab62c0b1c7/dacbbff1-3783-4e73-aa71-dbe41700eceb"
-					(reference "R406")
+					(reference "R407")
 					(unit 1)
 				)
@@
 	)
 	(symbol
+		(lib_id "Device:R")
+		(at 359.41 48.26 0)
+		(unit 1)
+		(exclude_from_sim no)
+		(in_bom yes)
+		(on_board yes)
+		(dnp no)
+		(property "Reference" "R405"
+			(at 359.41 50.8 90)
+			(effects
+				(font
+					(size 1.27 1.27)
+				)
+				(justify left)
+			)
+		)
+		(property "Value" "2K2"
+			(at 357.505 50.165 90)
+			(effects
+				(font
+					(size 1.27 1.27)
+				)
+				(justify left)
+			)
+		)
+		(property "Footprint" "Resistor_SMD:R_1206_3216Metric_Pad1.30x1.75mm_HandSolder"
+			(at 357.632 48.26 90)
+			(effects
+				(font
+					(size 1.27 1.27)
+				)
+				(hide yes)
+			)
+		)
+		(property "Datasheet" "~"
+			(at 359.41 48.26 0)
+			(effects
+				(font
+					(size 1.27 1.27)
+				)
+				(hide yes)
+			)
+		)
+		(property "Description" ""
+			(at 359.41 48.26 0)
+			(effects
+				(font
+					(size 1.27 1.27)
+				)
+			)
+		)
+		(property "Manufacturer_Name" "Yageo"
+			(at 359.41 48.26 90)
+			(effects
+				(font
+					(size 1.27 1.27)
+				)
+				(hide yes)
+			)
+		)
+		(property "Manufacturer_Part_Number" "RT1206FRE072K2L"
+			(at 359.41 48.26 90)
+			(effects
+				(font
+					(size 1.27 1.27)
+				)
+				(hide yes)
+			)
+		)
+		(pin "1"
+		)
+		(pin "2"
+		)
+		(instances
+			(project "raven"
+				(path "/af55e73e-5814-45b4-ac5c-0bab62c0b1c7/dacbbff1-3783-4e73-aa71-dbe41700eceb"
+					(reference "R405")
+					(unit 1)
+				)
+			)
+		)
+	)
+	(symbol
 		(lib_id "power:+5V")
 		(at 286.385 129.54 0)
@@
 		(on_board yes)
 		(dnp no)
-		(property "Reference" "R408"
+		(property "Reference" "R409"
 			(at 344.17 217.805 90)
 			(effects
@@
 			(project "raven"
 				(path "/af55e73e-5814-45b4-ac5c-0bab62c0b1c7/dacbbff1-3783-4e73-aa71-dbe41700eceb"
-					(reference "R408")
+					(reference "R409")
 					(unit 1)
 				)

Commit message: cosmetic
Other:
- moved on the sheet: C415
Changed lines of the file:
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@@
 	)
 	(junction
+		(at 171.45 270.51)
+		(diameter 0)
+		(color 0 0 0 0)
+	)
+	(junction
 		(at 56.515 73.66)
 		(diameter 0)
@@
 		(color 0 0 0 0)
 	)
-	(junction
-		(at 171.45 271.78)
-		(diameter 0)
-		(color 0 0 0 0)
-	)
 	(no_connect
 		(at 441.96 203.2)
@@
 		)
 	)
+	(wire
+		(pts
+			(xy 171.45 270.51) (xy 171.45 273.05)
+		)
+		(stroke
+			(width 0)
+			(type default)
+		)
+	)
 	(bus
 		(pts
@@
 	(wire
 		(pts
-			(xy 171.45 271.78) (xy 171.45 273.05)
-		)
-		(stroke
-			(width 0)
-			(type default)
-		)
-	)
-	(wire
-		(pts
 			(xy 467.995 124.46) (xy 470.535 124.46)
 		)
@@
 	(wire
 		(pts
-			(xy 187.96 271.78) (xy 194.945 271.78)
+			(xy 184.15 270.51) (xy 189.865 270.51)
 		)
 		(stroke
@@
 	(wire
 		(pts
-			(xy 194.945 271.78) (xy 194.945 272.415)
+			(xy 189.865 270.51) (xy 189.865 271.145)
 		)
 		(stroke
@@
 	(wire
 		(pts
-			(xy 171.45 271.78) (xy 182.88 271.78)
+			(xy 171.45 270.51) (xy 179.07 270.51)
 		)
 		(stroke
@@
 	(wire
 		(pts
-			(xy 171.45 269.24) (xy 171.45 271.78)
+			(xy 171.45 269.24) (xy 171.45 270.51)
 		)
 		(stroke
@@
 		(dnp no)
 		(property "Reference" "C404"
-			(at 126.365 77.47 90)
+			(at 129.54 75.946 90)
 			(effects
 				(font
@@
 		)
 		(property "Value" "0.1u"
-			(at 133.35 77.47 90)
+			(at 129.54 81.534 90)
 			(effects
 				(font
@@
 		(on_board yes)
 		(dnp no)
-		(fields_autoplaced yes)
 		(property "Reference" "U407"
-			(at 184.15 278.0598 0)
+			(at 166.37 274.574 0)
 			(effects
 				(font
@@
 		)
 		(property "Value" "24AA02E48"
-			(at 184.15 280.5998 0)
+			(at 178.054 291.084 0)
 			(effects
 				(font
@@
 	(symbol
 		(lib_id "power:GND")
-		(at 194.945 272.415 0)
+		(at 189.865 271.145 0)
 		(unit 1)
 		(exclude_from_sim no)
@@
 		(dnp no)
 		(property "Reference" "#PWR0458"
-			(at 194.945 278.765 0)
+			(at 189.865 277.495 0)
 			(effects
 				(font
@@
 		)
 		(property "Value" "GND"
-			(at 194.945 276.225 0)
+			(at 189.865 274.955 0)
 			(effects
 				(font
@@
 		)
 		(property "Footprint" ""
-			(at 194.945 272.415 0)
+			(at 189.865 271.145 0)
 			(effects
 				(font
@@
 		)
 		(property "Datasheet" ""
-			(at 194.945 272.415 0)
+			(at 189.865 271.145 0)
 			(effects
 				(font
@@
 		)
 		(property "Description" ""
-			(at 194.945 272.415 0)
+			(at 189.865 271.145 0)
 			(effects
 				(font
@@
 		(dnp no)
 		(property "Reference" "C408"
-			(at 294.005 163.83 90)
+			(at 297.18 162.306 90)
 			(effects
 				(font
@@
 		)
 		(property "Value" "0.1u"
-			(at 300.99 163.83 90)
+			(at 297.18 167.894 90)
 			(effects
 				(font
@@
 		(lib_name "c_100nf_smd1206_1")
 		(lib_id "68k:c_100nf_smd1206")
-		(at 185.42 271.78 270)
+		(at 181.61 270.51 270)
 		(unit 1)
 		(exclude_from_sim no)
@@
 		(dnp no)
 		(property "Reference" "C415"
-			(at 181.61 270.51 90)
+			(at 181.61 267.716 90)
 			(effects
 				(font
@@
 		)
 		(property "Value" "0.1u"
-			(at 188.595 270.51 90)
+			(at 181.61 273.558 90)
 			(effects
 				(font
@@
 		)
 		(property "Footprint" "Capacitor_SMD:C_1206_3216Metric_Pad1.33x1.80mm_HandSolder"
-			(at 160.02 265.43 0)
+			(at 156.21 264.16 0)
 			(effects
 				(font
@@
 		)
 		(property "Datasheet" "https://www.mouser.se/datasheet/2/447/KEM_C1002_X7R_SMD-3316098.pdf"
-			(at 162.56 271.78 0)
+			(at 158.75 270.51 0)
 			(effects
 				(font
@@
 		)
 		(property "Description" ""
-			(at 185.42 271.78 0)
+			(at 181.61 270.51 0)
 			(effects
 				(font
@@
 		)
 		(property "Manufacturer_Name" "Kemet"
-			(at 167.64 237.49 0)
+			(at 163.83 236.22 0)
 			(effects
 				(font
@@
 		)
 		(property "Manufacturer_Part_Number" "C1206C104K5RACTU"
-			(at 165.1 243.84 0)
+			(at 161.29 242.57 0)
 			(effects
 				(font

Commit message: A2: cosmetics and bom preparations
Parts:
- U402: value ATF22V10C-10PU -> ATF22V10
- U404: value MAX3245CAI+T -> MAX3245

Commit message: A2: bom
Parts:
- J401: Manufacturer_Name Wurth -> Wurth Elektronik
- U401, U403: Manufacturer_Name NXP -> Motorola
Changed lines of the file:
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@@
 			)
 		)
-		(property "Manufacturer_Name" "Wurth"
+		(property "Manufacturer_Name" "Wurth Elektronik"
 			(at 90.17 191.135 0)
 			(effects
@@
 			)
 		)
-		(property "Manufacturer_Name" "NXP"
+		(property "Manufacturer_Name" "Motorola"
 			(at 264.795 90.17 0)
 			(effects
@@
 			)
 		)
-		(property "Manufacturer_Name" "NXP"
+		(property "Manufacturer_Name" "Motorola"
 			(at 448.945 78.74 0)
 			(effects
