File: hw/raven/a2/raven.kicad_sch (KiCad schematic)
At the start: 72 parts, among them J101 Pinhdr_01x02, J102 JTAG IN, J103 Pinhdr_01x03, SW101 SW_Push, U101 74LS148, U102 74AHC157, U103 SN74LVCH16245, U104 MC68150, U105 CY2308, U106 SN74LVCH16245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

Commit message: cosmetic
Other:
- note added: "CPU interrupt trigger + startup config"
- note removed: "CPU interrupt triggger + startup config"
Changed lines of the file:
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@@
 		)
 	)
-	(text "CPU interrupt triggger + startup config"
+	(text "CPU interrupt trigger + startup config"
 		(exclude_from_sim no)
 		(at 358.14 21.59 0)
@@
 		)
 	)
-	(text_box "Changes from rev.A1:\nThis signal is now wire-or of IOCS16 and MEMCS16\n"
-		(exclude_from_sim no)
-		(at 730.25 391.795 0)
-		(size 27.94 8.255)
-		(margins 0.9525 0.9525 0.9525 0.9525)
-		(stroke
-			(width 0)
-			(type dot)
-		)
-		(fill
-			(type none)
-		)
-		(effects
-			(font
-				(size 1.27 1.27)
-			)
-			(justify left top)
-		)
-	)
 	(text_box "TEA / TRA:\nThe current slave asserts this input signal to indicate an error condition for the current transfer to immediately terminate the bus cycle. The assertion of TEA has precedence over TRA\nand TA for native-MC68060-style acknowledgment termination.\nFor MC68040-style acknowledge termination, TEA must be asserted with TA negated to\ncause the current bus cycle to immediately terminate with a bus error indication. For\nMC68040-style acknowledge termination, TRA must be held negated."
 		(exclude_from_sim no)
@@
 		(dnp no)
 		(property "Reference" "C102"
-			(at 294.64 36.83 90)
+			(at 297.18 35.814 90)
 			(effects
 				(font
@@
 		)
 		(property "Value" "0.1u"
-			(at 300.99 36.83 90)
+			(at 297.18 41.656 90)
 			(effects
 				(font
@@
 		(dnp no)
 		(property "Reference" "C101"
-			(at 434.34 34.925 90)
+			(at 436.88 34.036 90)
 			(effects
 				(font
@@
 		)
 		(property "Value" "0.1u"
-			(at 440.69 34.925 90)
+			(at 436.88 39.878 90)
 			(effects
 				(font
@@
 		(dnp no)
 		(property "Reference" "X101"
-			(at 36.83 116.84 0)
+			(at 37.084 116.84 0)
 			(effects
 				(font
@@
 		(dnp no)
 		(property "Reference" "U102"
-			(at 424.815 41.91 0)
+			(at 423.926 41.656 0)
 			(effects
 				(font

Commit message: A2: cosmetics and bom preparations
Parts:
- J101: value Pinhdr_01x02 -> PinHdr_01x02
- J102: value JTAG IN -> PinHdr_02x05
- SW101: value SW_Push -> Button
- U101: Manufacturer_Name TI -> Texas Instruments

Commit message: A2: bom
Parts:
- J103: value Pinhdr_01x03 -> PinHdr_01x03
- U103, U106: Manufacturer_Name NXP -> Nexperia
- U104: Manufacturer_Part_Number MC68150 -> MC68150FN40
- U107: Manufacturer_Part_Number MC68060 -> MC68060RC50
Changed lines of the file:
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@@
 			)
 		)
-		(property "Manufacturer_Name" "NXP"
+		(property "Manufacturer_Name" "Nexperia"
 			(at 585.47 156.845 0)
 			(effects
@@
 			)
 		)
-		(property "Value" "Pinhdr_01x03"
+		(property "Value" "PinHdr_01x03"
 			(at 786.003 291.465 0)
 			(effects
@@
 			)
 		)
-		(property "Manufacturer_Name" "NXP"
+		(property "Manufacturer_Name" "Nexperia"
 			(at 585.47 86.36 0)
 			(effects
@@
 			)
 		)
-		(property "Manufacturer_Part_Number" "MC68150"
+		(property "Manufacturer_Part_Number" "MC68150FN40"
 			(at 732.155 92.075 0)
 			(effects
@@
 			)
 		)
-		(property "Manufacturer_Part_Number" "MC68060"
+		(property "Manufacturer_Part_Number" "MC68060RC50"
 			(at 240.665 309.88 0)
 			(effects

Commit message: A2: minor clarifications
Changed lines of the file:
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@@
 		)
 	)
-	(global_label "PA[0..31]"
+	(global_label "PA[0..1]"
 		(shape bidirectional)
 		(at 755.015 73.025 0)
@@
 		)
 		(property "Intersheetrefs" "${INTERSHEET_REFS}"
-			(at 768.0016 73.025 0)
+			(at 766.7921 73.025 0)
 			(effects
 				(font
