File: hw/simm/rom_PLCC/simm72_rom_2M55.kicad_sch (KiCad schematic)
At the start: 9 parts, among them J1 SIMM72, U1 SST39LF040, U2 SST39LF040, U3 SST39LF040, U4 SST39LF040

Commit message: some restructuring of simm folders
Size shouldn't be in the folder and filenames since it depends on what chips one populates.
Added SMD rev.A1 with fixes to make it compatible with BYTE/WORD selectable nor flash (pin47 tied to VCC for WORD mode)
Other:
- title: Raven 2MB ROM -> Raven PLCC ROM
Changed lines of the file:
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@@
   (paper "A4")
   (title_block
-    (title "Raven 2MB ROM")
+    (title "Raven PLCC ROM")
     (date "2023")
     (rev "A0")
@@
     (pin "9")
     (instances
-      (project "simm72_rom_2M55"
+      (project "simm72_rom_plcc"
         (path "/0981ba96-97e1-483d-834d-af22b04cbe88"
           (reference "J1") (unit 1)
@@
     (pin "1")
     (instances
-      (project "simm72_rom_2M55"
+      (project "simm72_rom_plcc"
         (path "/0981ba96-97e1-483d-834d-af22b04cbe88"
           (reference "#PWR011") (unit 1)
@@
     (pin "1")
     (instances
-      (project "simm72_rom_2M55"
+      (project "simm72_rom_plcc"
         (path "/0981ba96-97e1-483d-834d-af22b04cbe88"
           (reference "#PWR02") (unit 1)
@@
     (pin "1")
     (instances
-      (project "simm72_rom_2M55"
+      (project "simm72_rom_plcc"
         (path "/0981ba96-97e1-483d-834d-af22b04cbe88"
           (reference "#PWR012") (unit 1)
@@
     (pin "1")
     (instances
-      (project "simm72_rom_2M55"
+      (project "simm72_rom_plcc"
         (path "/0981ba96-97e1-483d-834d-af22b04cbe88"
           (reference "#PWR07") (unit 1)
@@
     (pin "8")
     (instances
-      (project "simm72_rom_2M55"
+      (project "simm72_rom_plcc"
         (path "/0981ba96-97e1-483d-834d-af22b04cbe88"
           (reference "U3") (unit 1)
@@
     (pin "2")
     (instances
-      (project "simm72_rom_2M55"
+      (project "simm72_rom_plcc"
         (path "/0981ba96-97e1-483d-834d-af22b04cbe88"
           (reference "C4") (unit 1)
@@
     (pin "2")
     (instances
-      (project "simm72_rom_2M55"
+      (project "simm72_rom_plcc"
         (path "/0981ba96-97e1-483d-834d-af22b04cbe88"
           (reference "C2") (unit 1)
@@
     (pin "1")
     (instances
-      (project "simm72_rom_2M55"
+      (project "simm72_rom_plcc"
         (path "/0981ba96-97e1-483d-834d-af22b04cbe88"
           (reference "#PWR01") (unit 1)
@@
     (pin "1")
     (instances
-      (project "simm72_rom_2M55"
+      (project "simm72_rom_plcc"
         (path "/0981ba96-97e1-483d-834d-af22b04cbe88"
           (reference "#PWR05") (unit 1)
@@
     (pin "1")
     (instances
-      (project "simm72_rom_2M55"
+      (project "simm72_rom_plcc"
         (path "/0981ba96-97e1-483d-834d-af22b04cbe88"
           (reference "#PWR03") (unit 1)
@@
     (pin "8")
     (instances
-      (project "simm72_rom_2M55"
+      (project "simm72_rom_plcc"
         (path "/0981ba96-97e1-483d-834d-af22b04cbe88"
           (reference "U2") (unit 1)
@@
     (pin "2")
     (instances
-      (project "simm72_rom_2M55"
+      (project "simm72_rom_plcc"
         (path "/0981ba96-97e1-483d-834d-af22b04cbe88"
           (reference "C3") (unit 1)
@@
     (pin "8")
     (instances
-      (project "simm72_rom_2M55"
+      (project "simm72_rom_plcc"
         (path "/0981ba96-97e1-483d-834d-af22b04cbe88"
           (reference "U4") (unit 1)
@@
     (pin "1")
     (instances
-      (project "simm72_rom_2M55"
+      (project "simm72_rom_plcc"
         (path "/0981ba96-97e1-483d-834d-af22b04cbe88"
           (reference "#PWR014") (unit 1)
@@
     (pin "1")
     (instances
-      (project "simm72_rom_2M55"
+      (project "simm72_rom_plcc"
         (path "/0981ba96-97e1-483d-834d-af22b04cbe88"
           (reference "#PWR010") (unit 1)
@@
     (pin "1")
     (instances
-      (project "simm72_rom_2M55"
+      (project "simm72_rom_plcc"
         (path "/0981ba96-97e1-483d-834d-af22b04cbe88"
           (reference "#PWR08") (unit 1)
@@
     (pin "1")
     (instances
-      (project "simm72_rom_2M55"
+      (project "simm72_rom_plcc"
         (path "/0981ba96-97e1-483d-834d-af22b04cbe88"
           (reference "#PWR06") (unit 1)
@@
     (pin "2")
     (instances
-      (project "simm72_rom_2M55"
+      (project "simm72_rom_plcc"
         (path "/0981ba96-97e1-483d-834d-af22b04cbe88"
           (reference "C1") (unit 1)
@@
     (pin "1")
     (instances
-      (project "simm72_rom_2M55"
+      (project "simm72_rom_plcc"
         (path "/0981ba96-97e1-483d-834d-af22b04cbe88"
           (reference "#PWR04") (unit 1)
@@
     (pin "8")
     (instances
-      (project "simm72_rom_2M55"
+      (project "simm72_rom_plcc"
         (path "/0981ba96-97e1-483d-834d-af22b04cbe88"
           (reference "U1") (unit 1)
@@
     (pin "1")
     (instances
-      (project "simm72_rom_2M55"
+      (project "simm72_rom_plcc"
         (path "/0981ba96-97e1-483d-834d-af22b04cbe88"
           (reference "#PWR013") (unit 1)
@@
     (pin "1")
     (instances
-      (project "simm72_rom_2M55"
+      (project "simm72_rom_plcc"
         (path "/0981ba96-97e1-483d-834d-af22b04cbe88"
           (reference "#PWR09") (unit 1)
