File: hw/simm/rom_SMD/a0/simm72_rom_smd.kicad_sch (KiCad schematic)
At the start: 7 parts, among them IC1 SN74LVC2G08DCUR, IC2 SST39LFx01, IC3 SST39LFx01, J1 SIMM72

Commit message: some restructuring of simm folders
Size shouldn't be in the folder and filenames since it depends on what chips one populates.
Added SMD rev.A1 with fixes to make it compatible with BYTE/WORD selectable nor flash (pin47 tied to VCC for WORD mode)
Other:
- title: Raven 1MB ROM -> Raven SMD ROM
Changed lines of the file:
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@@
   (paper "A4")
   (title_block
-    (title "Raven 1MB ROM")
+    (title "Raven SMD ROM")
     (date "2023")
     (rev "A0")
@@
     (pin "9")
     (instances
-      (project "simm72_rom_1M55"
+      (project "simm72_rom_smd"
         (path "/0981ba96-97e1-483d-834d-af22b04cbe88"
           (reference "J1") (unit 1)
@@
     (pin "1")
     (instances
-      (project "simm72_rom_1M55"
+      (project "simm72_rom_smd"
         (path "/0981ba96-97e1-483d-834d-af22b04cbe88"
           (reference "#PWR02") (unit 1)
@@
     (pin "2")
     (instances
-      (project "simm72_rom_1M55"
+      (project "simm72_rom_smd"
         (path "/0981ba96-97e1-483d-834d-af22b04cbe88"
           (reference "C2") (unit 1)
@@
     (pin "1")
     (instances
-      (project "simm72_rom_1M55"
+      (project "simm72_rom_smd"
         (path "/0981ba96-97e1-483d-834d-af22b04cbe88"
           (reference "#PWR013") (unit 1)
@@
     (pin "1")
     (instances
-      (project "simm72_rom_1M55"
+      (project "simm72_rom_smd"
         (path "/0981ba96-97e1-483d-834d-af22b04cbe88"
           (reference "#PWR01") (unit 1)
@@
     (pin "1")
     (instances
-      (project "simm72_rom_1M55"
+      (project "simm72_rom_smd"
         (path "/0981ba96-97e1-483d-834d-af22b04cbe88"
           (reference "#PWR07") (unit 1)
@@
     (pin "1")
     (instances
-      (project "simm72_rom_1M55"
+      (project "simm72_rom_smd"
         (path "/0981ba96-97e1-483d-834d-af22b04cbe88"
           (reference "#PWR011") (unit 1)
@@
     (pin "1")
     (instances
-      (project "simm72_rom_1M55"
+      (project "simm72_rom_smd"
         (path "/0981ba96-97e1-483d-834d-af22b04cbe88"
           (reference "#PWR012") (unit 1)
@@
     (pin "3")
     (instances
-      (project "simm72_rom_1M55"
+      (project "simm72_rom_smd"
         (path "/0981ba96-97e1-483d-834d-af22b04cbe88"
           (reference "IC1") (unit 1)
@@
     (pin "1")
     (instances
-      (project "simm72_rom_1M55"
+      (project "simm72_rom_smd"
         (path "/0981ba96-97e1-483d-834d-af22b04cbe88"
           (reference "#PWR05") (unit 1)
@@
     (pin "1")
     (instances
-      (project "simm72_rom_1M55"
+      (project "simm72_rom_smd"
         (path "/0981ba96-97e1-483d-834d-af22b04cbe88"
           (reference "#PWR04") (unit 1)
@@
     (pin "2")
     (instances
-      (project "simm72_rom_1M55"
+      (project "simm72_rom_smd"
         (path "/0981ba96-97e1-483d-834d-af22b04cbe88"
           (reference "C3") (unit 1)
@@
     (pin "1")
     (instances
-      (project "simm72_rom_1M55"
+      (project "simm72_rom_smd"
         (path "/0981ba96-97e1-483d-834d-af22b04cbe88"
           (reference "#PWR03") (unit 1)
@@
     (pin "1")
     (instances
-      (project "simm72_rom_1M55"
+      (project "simm72_rom_smd"
         (path "/0981ba96-97e1-483d-834d-af22b04cbe88"
           (reference "#PWR010") (unit 1)
@@
     (pin "39")
     (instances
-      (project "simm72_rom_1M55"
+      (project "simm72_rom_smd"
         (path "/0981ba96-97e1-483d-834d-af22b04cbe88"
           (reference "IC2") (unit 1)
@@
     (pin "1")
     (instances
-      (project "simm72_rom_1M55"
+      (project "simm72_rom_smd"
         (path "/0981ba96-97e1-483d-834d-af22b04cbe88"
           (reference "#PWR06") (unit 1)
@@
     (pin "1")
     (instances
-      (project "simm72_rom_1M55"
+      (project "simm72_rom_smd"
         (path "/0981ba96-97e1-483d-834d-af22b04cbe88"
           (reference "#PWR08") (unit 1)
@@
     (pin "1")
     (instances
-      (project "simm72_rom_1M55"
+      (project "simm72_rom_smd"
         (path "/0981ba96-97e1-483d-834d-af22b04cbe88"
           (reference "#PWR09") (unit 1)
@@
     (pin "39")
     (instances
-      (project "simm72_rom_1M55"
+      (project "simm72_rom_smd"
         (path "/0981ba96-97e1-483d-834d-af22b04cbe88"
           (reference "IC3") (unit 1)
@@
     (pin "2")
     (instances
-      (project "simm72_rom_1M55"
+      (project "simm72_rom_smd"
         (path "/0981ba96-97e1-483d-834d-af22b04cbe88"
           (reference "C1") (unit 1)
