File: hw/simm/rom_SMD/a1/simm72_rom_smd.kicad_sch (KiCad schematic)
At the start: 7 parts, among them IC1 SN74LVC2G08DCUR, IC2 SST39LFx01, IC3 SST39LFx01, J1 SIMM72

Commit message: Update simm72_rom_smd.kicad_sch
Other:
- note added: "Changes from rev.A0 - Tied pin47 to vcc for compatibility with other manufacturers (selects WORD mode)"
- note added: "SST39LF400A SST39LF401C SST39LF402C SST39LF800A SST39LF801C SST39LF802C"
- note removed: "SST39LF401C SST39LF402C SST39LF801C SST39LF802C SST39LF400A SST39LF800A"
- moved on the sheet: C1, C2, C3, IC1, IC2, IC3, J1
