File: hw/raven/upgrades/ckbd/ckbd.kicad_pcb (KiCad board)
At the start: 4 copper layers, 35.6 x 39.4 mm, 19 parts, among them J103 USB, U101 CH559L, U102 74LVC1G34

Commit message: ckbd rev.d
Parts:
- removed U102: 74LVC1G34, Package_TO_SOT_SMD:SOT-23-5_HandSoldering
- added R107: 1K, Resistor_SMD:R_1206_3216Metric_Pad1.30x1.75mm_HandSolder, F.Cu at (111.0, 73.4)
- J103: footprint Connector_PinHeader_2.54mm:PinHeader_2x05_P2.54mm_Vertical -> 68k:USB2Header
- moved R101 6.17 mm to (111.0, 61.5)
- moved R102 5.79 mm to (111.0, 67.4)
Routing:
- net +5V: track 63.5 -> 73.8 mm
- net CLK4: track 4.97 -> 0.00 mm
- net FAN1: track 20.0 -> 23.8 mm
- net Net-(J104-Pin_4): track 3.80 -> 0.00 mm
- net GND: track 17.2 -> 15.0 mm, vias 11 -> 9
- net +3.3V: track 12.0 -> 10.8 mm, vias 6 -> 5
- net IKBD_TX: track 19.8 -> 19.2 mm, vias 1 -> 0
- net IKBD_RX: track 18.2 -> 18.7 mm, vias 1 -> 0
Other:
- board text added: "-##- program #--- uart-tx"
- board text added: "CKBD rev.d"
- board text removed: "---- int.osc --## ext.osc -##- program #--- uart-tx"
- board text removed: "CKBD rev.c"
