File: hw/raven/upgrades/ckbd/ckbd.kicad_sch (KiCad schematic)
At the start: 19 parts, among them J103 USB, U101 CH559L, U102 74LVC1G34

Commit message: ckbd rev.d
Parts:
- added R107: 1K, Resistor_SMD:R_1206_3216Metric_Pad1.30x1.75mm_HandSolder, symbol Device:R
- J103: footprint Connector_PinHeader_2.54mm:PinHeader_2x05_P2.54mm_Vertical -> 68k:USB2Header; symbol Connector_Generic:Conn_02x05_Odd_Even -> 68k:USB2Header
- U102: now not fitted; now left out of the parts list
Connections:
- net +5V: now also R107.1
- net FAN1: now also R107.2
- removed net key: J103.9 (Pin_9)
- no-connect marks 23 -> 22
Changed lines of the file:
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@@
 		(title "CKBD")
 		(date "2025")
-		(rev "c")
+		(rev "d")
 		(company "Licensed under CERN-OHL-W v2")
 		(comment 1 "(c)2025 Anders Granlund")
@@
 	)
 	(junction
+		(at 223.52 62.865)
+		(diameter 0)
+		(color 0 0 0 0)
+	)
+	(junction
 		(at 167.005 37.465)
 		(diameter 0)
@@
 	)
 	(no_connect
-		(at 325.755 167.005)
-	)
-	(no_connect
 		(at 320.675 76.835)
 	)
@@
 	(wire
 		(pts
+			(xy 223.52 59.69) (xy 223.52 62.865)
+		)
+		(stroke
+			(width 0)
+			(type default)
+		)
+	)
+	(wire
+		(pts
 			(xy 327.025 148.59) (xy 327.025 156.845)
 		)
@@
 	(wire
 		(pts
+			(xy 223.52 50.165) (xy 223.52 52.07)
+		)
+		(stroke
+			(width 0)
+			(type default)
+		)
+	)
+	(wire
+		(pts
 			(xy 167.005 37.465) (xy 167.005 42.545)
 		)
@@
 	(wire
 		(pts
-			(xy 201.295 62.865) (xy 205.105 62.865)
+			(xy 201.295 62.865) (xy 223.52 62.865)
 		)
 		(stroke
@@
 	(wire
 		(pts
-			(xy 325.755 167.005) (xy 329.565 167.005)
-		)
-		(stroke
-			(width 0)
-			(type default)
-		)
-	)
-	(wire
-		(pts
 			(xy 320.675 76.835) (xy 330.835 76.835)
 		)
@@
 	(wire
 		(pts
+			(xy 223.52 62.865) (xy 228.6 62.865)
+		)
+		(stroke
+			(width 0)
+			(type default)
+		)
+	)
+	(wire
+		(pts
 			(xy 81.915 114.935) (xy 81.915 116.205)
 		)
@@
 		)
 	)
-	(label "key"
-		(at 327.025 167.005 0)
-		(effects
-			(font
-				(size 1.27 1.27)
-			)
-			(justify left bottom)
-		)
-	)
 	(label "nc"
 		(at 342.265 167.005 0)
@@
 	(global_label "FAN1"
 		(shape output)
-		(at 205.105 62.865 0)
+		(at 228.6 62.865 0)
 		(fields_autoplaced yes)
 		(effects
@@
 		)
 		(property "Intersheetrefs" "${INTERSHEET_REFS}"
-			(at 211.1695 62.865 0)
+			(at 234.6645 62.865 0)
 			(effects
 				(font
@@
 		(at 57.15 182.88 0)
 		(unit 1)
-		(exclude_from_sim no)
-		(in_bom yes)
-		(on_board yes)
-		(dnp no)
+		(exclude_from_sim yes)
+		(in_bom no)
+		(on_board no)
+		(dnp yes)
 		(property "Reference" "U102"
 			(at 68.58 176.4598 0)
@@
 	)
 	(symbol
+		(lib_id "power:+5V")
+		(at 223.52 50.165 0)
+		(mirror y)
+		(unit 1)
+		(exclude_from_sim no)
+		(in_bom yes)
+		(on_board yes)
+		(dnp no)
+		(property "Reference" "#PWR0125"
+			(at 223.52 53.975 0)
+			(effects
+				(font
+					(size 1.27 1.27)
+				)
+				(hide yes)
+			)
+		)
+		(property "Value" "+5V"
+			(at 225.044 46.355 0)
+			(effects
+				(font
+					(size 1.27 1.27)
+				)
+				(justify left)
+			)
+		)
+		(property "Footprint" ""
+			(at 223.52 50.165 0)
+			(effects
+				(font
+					(size 1.27 1.27)
+				)
+				(hide yes)
+			)
+		)
+		(property "Datasheet" ""
+			(at 223.52 50.165 0)
+			(effects
+				(font
+					(size 1.27 1.27)
+				)
+				(hide yes)
+			)
+		)
+		(property "Description" "Power symbol creates a global label with name \"+5V\""
+			(at 223.52 50.165 0)
+			(effects
+				(font
+					(size 1.27 1.27)
+				)
+				(hide yes)
+			)
+		)
+		(pin "1"
+		)
+		(instances
+			(project "ckbd"
+				(path "/cd7a93ea-0fc9-4e8f-aeb2-c40a58c62e5f"
+					(reference "#PWR0125")
+					(unit 1)
+				)
+			)
+		)
+	)
+	(symbol
 		(lib_id "power:GND")
 		(at 161.925 130.175 0)
@@
 	)
 	(symbol
+		(lib_id "Device:R")
+		(at 223.52 55.88 0)
+		(unit 1)
+		(exclude_from_sim no)
+		(in_bom yes)
+		(on_board yes)
+		(dnp no)
+		(property "Reference" "R107"
+			(at 223.52 55.88 90)
+			(effects
+				(font
+					(size 1.27 1.27)
+				)
+			)
+		)
+		(property "Value" "1K"
+			(at 221.615 55.88 90)
+			(effects
+				(font
+					(size 1.27 1.27)
+				)
+			)
+		)
+		(property "Footprint" "Resistor_SMD:R_1206_3216Metric_Pad1.30x1.75mm_HandSolder"
+			(at 221.742 55.88 90)
+			(effects
+				(font
+					(size 1.27 1.27)
+				)
+				(hide yes)
+			)
+		)
+		(property "Datasheet" "~"
+			(at 223.52 55.88 0)
+			(effects
+				(font
+					(size 1.27 1.27)
+				)
+				(hide yes)
+			)
+		)
+		(property "Description" ""
+			(at 223.52 55.88 0)
+			(effects
+				(font
+					(size 1.27 1.27)
+				)
+			)
+		)
+		(property "Manufacturer_Name" "Yageo"
+			(at 223.52 55.88 0)
+			(effects
+				(font
+					(size 1.27 1.27)
+				)
+				(hide yes)
+			)
+		)
+		(property "Manufacturer_Part_Number" "RT1206FRE071KL"
+			(at 223.52 55.88 0)
+			(effects
+				(font
+					(size 1.27 1.27)
+				)
+				(hide yes)
+			)
+		)
+		(pin "1"
+		)
+		(pin "2"
+		)
+		(instances
+			(project "ckbd"
+				(path "/cd7a93ea-0fc9-4e8f-aeb2-c40a58c62e5f"
+					(reference "R107")
+					(unit 1)
+				)
+			)
+		)
+	)
+	(symbol
 		(lib_id "power:GND")
 		(at 142.875 38.735 0)
@@
 	)
 	(symbol
-		(lib_id "Connector_Generic:Conn_02x05_Odd_Even")
+		(lib_id "68k:USB2Header")
 		(at 334.645 161.925 0)
 		(unit 1)
@@
 			)
 		)
-		(property "Footprint" "Connector_PinHeader_2.54mm:PinHeader_2x05_P2.54mm_Vertical"
+		(property "Footprint" "68k:USB2Header"
 			(at 334.645 161.925 0)
 			(effects
@@
 		(pin "7"
 		)
-		(pin "9"
-		)
 		(pin "2"
